File: hardware/daughterboard/daughterboard.kicad_sch (KiCad schematic)
At the start: 87 parts, among them J1 Custom_PCIe_x4, U0 XTR200, U1 XTR200, U10 REF5030EIDR, U11 AD7193, U2 XTR200, U20 DAC80508Z, U3 XTR200, U4 XTR200, U5 XTR200, U6 XTR200, U7 XTR200, U8 SN74LV165

Commit message: add board
Parts:
- added FID1, FID2: Fiducial, Fiducial:Fiducial_1mm_Mask2mm, symbol Mechanical:Fiducial
- 3V3, CH0, CH1, CH2, CH3, CH4, CH5, CH6, CH7, DAC0, DAC1, DAC2, DAC3, DAC4, DAC5, DAC6, DAC7: value ~ -> (none)
Other:
- note added: "!padne VOLTAGE v=3.3 p=J1.A2 n=J1.B2 !padne VOLTAGE v=12 p=J1.A3 n=J1.A4 !padne RESISTANCE r=0.1 a=L1.1 b=L1.2 !padne RESISTANCE r=1.5 a=R27.2 b=R27.1 !padne CURRENT i=4mA f=U11.24 t=U11.22 !padne CURRENT i=1mA f=U11.25 t=U11.23 !padne CURRENT i=1mA f=U10.2 t=U10.4 !padne CURRENT i=3mA f=U20.7 t=U20.6 !padne CURRENT i=1mA f=U8.16 t=U8.8 ; CH0: U0 -> J1.A13/B13, load 800R to gnd finger A14, sense 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"
