File: hardware/daughterboard/daughterboard.kicad_sch (KiCad schematic)
At the start: 89 parts, among them J1 Custom_PCIe_x4, U0 XTR200, U1 XTR200, U10 REF5030EIDR, U11 AD7193, U2 XTR200, U20 DAC80508Z, U3 XTR200, U4 XTR200, U5 XTR200, U6 XTR200, U7 XTR200, U8 SN74LV165, U9 AT21CS01

Commit message: Rework AD7193 DVDD pi filter; resolve L1/R27 BOM TBDs
The DVDD filter (C17 - L1/R27 - C18) had all its local capacitance on the
unfiltered side: C22+C23+C17 = 1.2 uF on +3.3V, versus 100 nF on VDDA.

- Move C23 (1 uF) from +3.3V to VDDA. Zero BOM/placement change: it was
  already back-to-back with C18 at (87.50, 84.00). Filtered node goes
  100 nF -> 1.1 uF. Removed the stale +3.3V routing that ran through the
  pad, which would otherwise have shorted out L1 and R27.
- R27 1.5 -> 10 ohm. Corner 97 kHz -> 14 kHz for 4.2 mV drop; AD7193 DIDD
  is 0.4 mA (internal oscillator, no crystal fitted). Damping Q = 0.09.
- L1 resolved to C96708 (Sunlord GZ1608U601CTF, 600R@100MHz, 380 mohm,
  500 mA). The old "1.5 A" requirement was a phantom from the KiCad symbol
  name FerriteBead_0603_1.5A, not the design.
- R27 resolved to C144117 (YAGEO AF0603JR-0710RL, 10 ohm 5%).
- padne directives updated to match: r=10 on R27, r=0.38 on L1.
- Schematic note "Use NP0 for C17, C18" -> "Use X7R": 100 nF C0G does not
  exist in 0603 at 50 V, and these are supply shunts where C0G buys nothing.

master_bom_lcsc.csv (new file) additionally fixes:
- C9 was grouped on the 10 uF line but is 0.1 uF; moved to the 100 nF line.
  100 nF 152 -> 160 units, 10 uF 16 -> 8 units.
- R18 row had an unquoted comma splitting it into 18 CSV fields.
- Totals: 717.34 -> 717.70, LCSC 308.88 -> 307.38.

Co-Authored-By: Claude Opus 5 <noreply@anthropic.com>
Parts:
- C1, C10, C12, C14, C15, C17, C18, C19, C2, C20, C21, C22, C24, C3, C4, C5, C6, C7, C8: LCSC (none) -> C14663
- C11, C13, C16, C23: LCSC (none) -> C15849
- C25: LCSC (none) -> C96446
- C9: value 10uF -> 0.1uF; LCSC (none) -> C14663
- D1: LCSC (none) -> C125114
- L1: LCSC (none) -> C96708
- R1, R10, R11, R12, R2, R3, R4, R9: LCSC (none) -> C122538
- R13, R14, R15, R16, R5, R6, R7, R8: LCSC (none) -> C154077
- R17: value 100k -> 500; LCSC (none) -> C23179
- R18: LCSC (none) -> C13167
- R19, R20, R21, R22, R23, R24, R25, R26: LCSC (none) -> C513565
- R27: value 1.5 -> 10; LCSC (none) -> C144117
- U0, U1, U2, U3, U4, U5, U6, U7: LCSC (none) -> C52091642
- U10: value REF5030EIDR -> REF5030IDGKR; LCSC (none) -> C2862926
- U11: LCSC (none) -> C125128
- U20: value DAC80508Z -> DAC80508ZR; LCSC (none) -> C2679499
- U8: LCSC (none) -> C201716
- U9: LCSC (none) -> C616192
Connections:
- net +3.3V: no longer C23.1
- net GND: now also D1.1 (K); no longer D1.2 (A)
- net VDDA: now also C23.1
- net at R17.1: now also D1.2 (A); no longer D1.1 (K)
Other:
- note added: "; ============================================================================ ; padne directives - KOI 8x8 daughterboard ; rev: A30=+12V, C25 bulk, U9 AT21CS01, R18=2.7k ; 2026-07-30: C23 moved +3.3V -> VDDA (now 1.1uF on the filtered node); ; R27 1.5 -> 10 ohm; L1 DCR 0.1 -> 0.38 (Sunlord GZ1608U601CTF) ; All designators/pads verified against daughterboard.kicad_pcb ; ; v3 CHANGE: the optional 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"
- note added: "Best to use REF5030EIDR"
- note added: "Use X7R for C17, C18"
- note added: "Use capacitors above 16V CC0603KRX7R9BB104 - C14663 100nF 50V X7R ±10% 0603 Multilayer Ceramic Capacitors MLCC - SMD/SMT ROHS YAGEO RT0603BRD074K7L 4.7k -55℃~+155℃ 100mW 4.7kΩ 75V"
- note added: "XTR200"
- note removed: "; ============================================================================ ; padne directives - KOI 8x8 daughterboard ; rev: A30=+12V, C25 bulk, U9 AT21CS01, R18=2.7k ; All designators/pads verified against daughterboard.kicad_pcb ; ; v3 CHANGE: the optional DAC-trace block is disabled. In v2 it injected ; +50uA at the DAC pin and drew -50uA at the XTR pin of the SAME net, giving ; each DACx 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"
- note removed: "maybe move the power pins"
- moved on the sheet: C12, C13, C14, C17, C18, C21, C22, C23, CH0, CH1, CH2, CH3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

Commit message: OPA2333 sense buffers and XTR200 EF fault-detection chain
Two daughterboard revisions plus the firmware to drive them.

OPA2333 sense buffers (root-causes the 3 mV offset):
- The ~3 mV offset seen during the 8-board test was the AD7193's *internal*
  input buffer. With the 6:1 divider, a low-current channel's ADC input sits
  below the buffered mode's usable common-mode range, so the buffer added a
  systematic offset instead of tracking.
- Fixed by disabling it (CONF.BUF = 0) and adding 8 external unity-gain
  followers: U13-U16 (OPA2333, 2 ch per package) between the divider taps and
  the ADC inputs, with R28-R35 1k series and C26-C33 100nF anti-alias
  (corner 1.59 kHz; was 339 kHz at 100R/4.7nF, which attenuated neither the
  OPA333 chop nor the AD7193 modulator rate).

XTR200 EF fault detection:
- Each daughterboard's SN74LV165 (U8) samples its eight XTR200 EF pins; the
  motherboard daisy-chains all eight into one 64-bit register on a private
  bit-banged 3-wire bus (CP=GP16, Q7=GP17, PL=GP18), so reading it never
  disturbs SPI0 (ADC + '595) or SPI1 (DAC).
- New EFChain.cpp/.h; loop() polls every 20 ms, latches a new fault, zeroes
  that channel's DAC and pins it at 0 mA until FAULTCLR.
- New host commands: FAULT?, FAULTCLR, FAULTEN ON|OFF.
- Documented limits: EF is one shared flag (open / saturation / SET short /
  UVLO <8 V / >150 C); open detection only arms above IOUT ~0.75 mA with
  RSET = 4.7k; an unpopulated slot breaks the chain, so efValidMask() reports
  which boards' bits are trustworthy.

Also:
- master_bom_lcsc.csv: U13-U16 and R28-R35 rows added (both LCSC-TBD), 100nF
  line 160 -> 224 units for C26-C33. Total understated until the OPA2333 line
  is priced.
- README: 3 mV offset moved from open issue to resolved.
- motherboard.kicad_pcb: 64 further routed segments.
- padne_plots_layers.py: per-layer padne plotting helper.
- paper/todo.txt: working notes.

Co-Authored-By: Claude Opus 5 <noreply@anthropic.com>
Parts:
- added C26, C27, C28, C29, C30, C31, C32, C33: 100nF, Capacitor_SMD:C_0603_1608Metric, symbol Device:C_Small
- added R28, R29, R30, R31, R32, R33, R34, R35: 1k, Resistor_SMD:R_0603_1608Metric, symbol Device:R_Small_US
- added U13, U14, U15, U16: OPA2333xxDRB, Package_SON:Texas_S-PVSON-N8, symbol Amplifier_Operational:OPA2333xxDRB
- C1, C10, C12, C14, C15, C17, C18, C19, C2, C20, C21, C22, C24, C3, C4, C5, C6, C7, C8, C9: value 0.1uF -> 100nF
Connections:
- net +3.3V: now also U13.8 (V+), U14.8 (V+), U15.8 (V+), U16.8 (V+)
- net CH0_V: now also C26.1, R28.1; no longer R2.1, R6.2
- net CH1_V: now also C27.1, R29.1; no longer R10.1, R14.2
- net CH2_V: now also C28.1, R30.1; no longer R13.2, R9.1
- net CH3_V: now also C29.1, R31.1; no longer R1.1, R5.2
- net CH4_V: now also C30.1, R32.1; no longer R4.1, R8.2
- net CH5_V: now also C31.1, R33.1; no longer R12.1, R16.2
- net CH6_V: now also C32.1, R34.1; no longer R11.1, R15.2
- net CH7_V: now also C33.1, R35.1; no longer R3.1, R7.2
- net GND: now also C26.2, C27.2, C28.2, C29.2, C30.2, C31.2, C32.2, C33.2, U13.4 (V-), U13.9 (PAD), U14.4 (V-), U14.9 (PAD), U15.4 (V-), U15.9 (PAD), U16.4 (V-), U16.9 (PAD)
- new net: R29.2, U13.6 (-), U13.7
- new net: R34.2, U16.1, U16.2 (-)
- new net: R32.2, U15.1, U15.2 (-)
- new net: R30.2, U14.1, U14.2 (-)
- new net: R31.2, U14.6 (-), U14.7
- new net: R33.2, U15.6 (-), U15.7
- new net: R28.2, U13.1, U13.2 (-)
- new net: R35.2, U16.6 (-), U16.7
- new net CH0_B: R2.1, R6.2, U13.3 (+)
- new net CH1_B: R10.1, R14.2, U13.5 (+)
- new net CH2_B: R13.2, R9.1, U14.3 (+)
- new net CH3_B: R1.1, R5.2, U14.5 (+)
- new net CH4_B: R4.1, R8.2, U15.3 (+)
- new net CH5_B: R12.1, R16.2, U15.5 (+)
- new net CH6_B: R11.1, R15.2, U16.3 (+)
- new net CH7_B: R3.1, R7.2, U16.5 (+)
Other:
- note added: "; ============================================================================ ; padne directives - KOI 8x8 daughterboard ; rev: A30=+12V, C25 bulk, U9 AT21CS01, R18=2.7k ; 2026-07-30: C23 moved +3.3V -> VDDA (now 1.1uF on the filtered node); ; R27 1.5 -> 10 ohm; L1 DCR 0.1 -> 0.38 (Sunlord GZ1608U601CTF) ; 2026-08-05: OPA2333 input buffers U13-U16 added between the sense dividers ; and the AD719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"
- note added: "Buffers"
- note removed: "; ============================================================================ ; padne directives - KOI 8x8 daughterboard ; rev: A30=+12V, C25 bulk, U9 AT21CS01, R18=2.7k ; 2026-07-30: C23 moved +3.3V -> VDDA (now 1.1uF on the filtered node); ; R27 1.5 -> 10 ohm; L1 DCR 0.1 -> 0.38 (Sunlord GZ1608U601CTF) ; All designators/pads verified against daughterboard.kicad_pcb ; ; v3 CHANGE: the optional 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"
- note removed: "LEDs"
- note removed: "Notes"
- moved on the sheet: 3V3, C12, C13, C20, C21, C24, C25, D1, FID1, FID2, R17, R18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

Commit message: hardware: release both boards to fabrication
Fab outputs regenerated from the current designs and sent out 2026-08-12.

Motherboard:
- +12V sense divider R5/R10 (100k/22k) + C10 filter at the Pico ADC pin
  -> GPIO26/ADC0, ratio 0.1803
- U3.~OE cut over from hardwired GND to GPIO19 (R9 10k pull-up)
- D2 SMBJ13A -> SMBJ16A (13 V standoff conducts on a 15 V rail)
- D6 gate-source clamp fixed at BZT52C18 (C192739)
- J1..J8.B31 tied to GND on all eight; dangling one-node PRSNT net deleted

Daughterboard:
- 1k series resistors R28-R35 into the OPA2333 followers
- L1 ferrite requoted C96708 (delisted) -> C133937, same 600R@100MHz
- U10 REF5030IDGKR -> REF5030EIDR; test points and the card edge J1 taken
  out of the BOM (bare pads / edge fingers, not parts)

master_bom.csv: D2 requote, D6/C10/R5/R10 added, L1 priced; $709.08 -> $709.29.
POWER.md: production/ is no longer stale (it is the released set); the two
remaining open items are schematic-drawing hygiene, not connectivity.
README: status section reflects the boards being in fab.

Co-Authored-By: Claude Opus 5 <noreply@anthropic.com>
Parts:
- 3V3, CH0, CH1, CH2, CH3, CH4, CH5, CH6, CH7, DAC0, DAC1, DAC2, DAC3, DAC4, DAC5, DAC6, DAC7, J1: now left out of the parts list
- L1: LCSC C96708 -> C133937; Part Number MI0603K300R-10 -> FCM1608KF-601T05
- R28, R29, R30, R31, R32, R33, R34, R35: LCSC (none) -> C22548
- U10: value REF5030IDGKR -> REF5030EIDR; LCSC C2862926 -> (none)
- U11: LCSC C125128 -> (none)
Changed lines of the file:
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@@
 		(body_style 1)
 		(exclude_from_sim no)
-		(in_bom yes)
+		(in_bom no)
 		(on_board yes)
 		(in_pos_files yes)
@@
 			)
 		)
-		(property "LCSC" "C125128"
+		(property "LCSC" ""
 			(at 127 217.17 0)
 			(hide yes)
@@
 		(body_style 1)
 		(exclude_from_sim no)
-		(in_bom yes)
+		(in_bom no)
 		(on_board yes)
 		(in_pos_files yes)
@@
 		(body_style 1)
 		(exclude_from_sim no)
-		(in_bom yes)
+		(in_bom no)
 		(on_board yes)
 		(in_pos_files yes)
@@
 			)
 		)
-		(property "LCSC" ""
+		(property "LCSC" "C22548"
 			(at 316.23 74.93 0)
 			(hide yes)
@@
 		(body_style 1)
 		(exclude_from_sim no)
-		(in_bom yes)
+		(in_bom no)
 		(on_board yes)
 		(in_pos_files yes)
@@
 		(body_style 1)
 		(exclude_from_sim no)
-		(in_bom yes)
+		(in_bom no)
 		(on_board yes)
 		(in_pos_files yes)
@@
 			)
 		)
-		(property "LCSC" ""
+		(property "LCSC" "C22548"
 			(at 378.46 118.11 0)
 			(hide yes)
@@
 		(body_style 1)
 		(exclude_from_sim no)
-		(in_bom yes)
+		(in_bom no)
 		(on_board yes)
 		(in_pos_files yes)
@@
 			)
 		)
-		(property "LCSC" ""
+		(property "LCSC" "C22548"
 			(at 316.23 118.11 0)
 			(hide yes)
@@
 			)
 		)
-		(property "LCSC" ""
+		(property "LCSC" "C22548"
 			(at 378.46 74.93 0)
 			(hide yes)
@@
 			)
 		)
-		(property "Value" "REF5030IDGKR"
+		(property "Value" "REF5030EIDR"
 			(at 125.3333 38.1 0)
 			(show_name no)
@@
 			)
 		)
-		(property "LCSC" "C2862926"
+		(property "LCSC" ""
 			(at 125.73 45.72 0)
 			(hide yes)
@@
 			)
 		)
-		(property "Part Number" "MI0603K300R-10"
+		(property "Part Number" "FCM1608KF-601T05"
 			(at 137.922 267.97 0)
 			(hide yes)
@@
 			)
 		)
-		(property "LCSC" "C96708"
+		(property "LCSC" "C133937"
 			(at 127 265.43 90)
 			(hide yes)
@@
 			)
 		)
-		(property "LCSC" ""
+		(property "LCSC" "C22548"
 			(at 316.23 147.32 0)
 			(hide yes)
@@
 		(body_style 1)
 		(exclude_from_sim no)
-		(in_bom yes)
+		(in_bom no)
 		(on_board yes)
 		(in_pos_files yes)
@@
 		(body_style 1)
 		(exclude_from_sim no)
-		(in_bom yes)
+		(in_bom no)
 		(on_board yes)
 		(in_pos_files yes)
@@
 		(body_style 1)
 		(exclude_from_sim no)
-		(in_bom yes)
+		(in_bom no)
 		(on_board yes)
 		(in_pos_files yes)
@@
 		(body_style 1)
 		(exclude_from_sim no)
-		(in_bom yes)
+		(in_bom no)
 		(on_board yes)
 		(in_pos_files yes)
@@
 			)
 		)
-		(property "LCSC" ""
+		(property "LCSC" "C22548"
 			(at 378.46 45.72 0)
 			(hide yes)
@@
 			)
 		)
-		(property "LCSC" ""
+		(property "LCSC" "C22548"
 			(at 316.23 45.72 0)
 			(hide yes)
@@
 			)
 		)
-		(property "LCSC" ""
+		(property "LCSC" "C22548"
 			(at 378.46 147.32 0)
 			(hide yes)
@@
 		(body_style 1)
 		(exclude_from_sim no)
-		(in_bom yes)
+		(in_bom no)
 		(on_board yes)
 		(in_pos_files yes)
@@
 		(body_style 1)
 		(exclude_from_sim no)
-		(in_bom yes)
+		(in_bom no)
 		(on_board yes)
 		(in_pos_files yes)
@@
 		(body_style 1)
 		(exclude_from_sim no)
-		(in_bom yes)
+		(in_bom no)
 		(on_board yes)
 		(in_pos_files yes)
@@
 		(body_style 1)
 		(exclude_from_sim no)
-		(in_bom yes)
+		(in_bom no)
 		(on_board yes)
 		(in_pos_files yes)
@@
 		(body_style 1)
 		(exclude_from_sim no)
-		(in_bom yes)
+		(in_bom no)
 		(on_board yes)
 		(in_pos_files yes)
@@
 		(body_style 1)
 		(exclude_from_sim no)
-		(in_bom yes)
+		(in_bom no)
 		(on_board yes)
 		(in_pos_files yes)
@@
 		(body_style 1)
 		(exclude_from_sim no)
-		(in_bom yes)
+		(in_bom no)
 		(on_board yes)
 		(in_pos_files yes)
@@
 		(body_style 1)
 		(exclude_from_sim no)
-		(in_bom yes)
+		(in_bom no)
 		(on_board yes)
 		(in_pos_files yes)
