File: hardware/daughterboard/daughterboard.kicad_pcb (KiCad board)
At the start: 4 copper layers, 51 x 51 mm, 112 parts, among them J1 Custom_PCIe_x4, U0 XTR200, U1 XTR200, U10 REF5030IDGKR, U11 AD7193, U13 OPA2333xxDRB, U14 OPA2333xxDRB, U15 OPA2333xxDRB, U16 OPA2333xxDRB, U2 XTR200, U20 DAC80508ZR, U3 XTR200, U4 XTR200, U5 XTR200, U6 XTR200, U7 XTR200, U8 SN74LV165, U9 AT21CS01

Commit message: hardware: release both boards to fabrication
Fab outputs regenerated from the current designs and sent out 2026-08-12.

Motherboard:
- +12V sense divider R5/R10 (100k/22k) + C10 filter at the Pico ADC pin
  -> GPIO26/ADC0, ratio 0.1803
- U3.~OE cut over from hardwired GND to GPIO19 (R9 10k pull-up)
- D2 SMBJ13A -> SMBJ16A (13 V standoff conducts on a 15 V rail)
- D6 gate-source clamp fixed at BZT52C18 (C192739)
- J1..J8.B31 tied to GND on all eight; dangling one-node PRSNT net deleted

Daughterboard:
- 1k series resistors R28-R35 into the OPA2333 followers
- L1 ferrite requoted C96708 (delisted) -> C133937, same 600R@100MHz
- U10 REF5030IDGKR -> REF5030EIDR; test points and the card edge J1 taken
  out of the BOM (bare pads / edge fingers, not parts)

master_bom.csv: D2 requote, D6/C10/R5/R10 added, L1 priced; $709.08 -> $709.29.
POWER.md: production/ is no longer stale (it is the released set); the two
remaining open items are schematic-drawing hygiene, not connectivity.
README: status section reflects the boards being in fab.

Co-Authored-By: Claude Opus 5 <noreply@anthropic.com>
Parts:
- C1, C10, C12, C14, C15, C17, C18, C19, C2, C20, C21, C22, C24, C3, C4, C5, C6, C7, C8, C9: value 0.1uF -> 100nF
- U10: value REF5030IDGKR -> REF5030EIDR
- renumbered VREF to VREF1
Routing:
- net +12V: track 115.4 -> 114.9 mm
Changed lines of the file:
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@@
 			)
 		)
-		(property "Value" "0.1uF"
+		(property "Value" "100nF"
 			(at 0 1.43 90)
 			(layer "F.Fab")
@@
 			)
 		)
-		(property "Value" "REF5030IDGKR"
+		(property "Value" "REF5030EIDR"
 			(at 0 3.4 0)
 			(layer "F.Fab")
@@
 			)
 		)
-		(property "LCSC" "C2862926"
+		(property "LCSC" ""
 			(at 0 0 180)
 			(unlocked yes)
@@
 			)
 		)
-		(property "Value" "0.1uF"
+		(property "Value" "100nF"
 			(at 0 1.43 0)
 			(layer "F.Fab")
@@
 			)
 		)
+		(attr exclude_from_bom)
 		(duplicate_pad_numbers_are_jumpers no)
 		(fp_circle
@@
 			)
 		)
+		(attr exclude_from_bom)
 		(duplicate_pad_numbers_are_jumpers no)
 		(fp_circle
@@
 			)
 		)
-		(property "Value" "0.1uF"
+		(property "Value" "100nF"
 			(at 0 1.43 90)
 			(layer "F.Fab")
@@
 			)
 		)
-		(property "Value" "0.1uF"
+		(property "Value" "100nF"
 			(at 0 1.43 0)
 			(layer "F.Fab")
@@
 			)
 		)
-		(property "Value" "0.1uF"
+		(property "Value" "100nF"
 			(at 0 1.43 90)
 			(layer "F.Fab")
@@
 			)
 		)
+		(attr exclude_from_bom)
 		(duplicate_pad_numbers_are_jumpers no)
 		(fp_line
@@
 			)
 		)
+		(attr exclude_from_bom)
 		(duplicate_pad_numbers_are_jumpers no)
 		(fp_circle
@@
 			)
 		)
+		(attr exclude_from_bom)
 		(duplicate_pad_numbers_are_jumpers no)
 		(fp_circle
@@
 			)
 		)
-		(property "Value" "0.1uF"
+		(property "Value" "100nF"
 			(at 0 1.43 0)
 			(layer "F.Fab")
@@
 			)
 		)
+		(attr exclude_from_bom)
 		(duplicate_pad_numbers_are_jumpers no)
 		(fp_circle
@@
 			)
 		)
-		(property "Value" "0.1uF"
+		(property "Value" "100nF"
 			(at 0 1.43 0)
 			(layer "F.Fab")
@@
 			)
 		)
+		(attr exclude_from_bom)
 		(duplicate_pad_numbers_are_jumpers no)
 		(fp_circle
@@
 			)
 		)
-		(property "Value" "0.1uF"
+		(property "Value" "100nF"
 			(at 0 1.43 0)
 			(layer "F.Fab")
@@
 		(descr "SMD pad as test Point, diameter 1.0mm")
 		(tags "test point SMD pad")
-		(property "Reference" "VREF"
+		(property "Reference" "VREF1"
 			(at -3.3 1 0)
 			(layer "F.SilkS")
@@
 			)
 		)
+		(attr exclude_from_bom)
 		(duplicate_pad_numbers_are_jumpers no)
 		(fp_circle
@@
 			)
 		)
-		(property "LCSC" "C125128"
+		(property "LCSC" ""
 			(at 0 0 180)
 			(unlocked yes)
@@
 			)
 		)
-		(property "Value" "0.1uF"
+		(property "Value" "100nF"
 			(at 0 1.43 0)
 			(layer "F.Fab")
@@
 			)
 		)
+		(attr exclude_from_bom)
 		(duplicate_pad_numbers_are_jumpers no)
 		(fp_circle
@@
 			)
 		)
+		(attr exclude_from_bom)
 		(duplicate_pad_numbers_are_jumpers no)
 		(fp_circle
@@
 			)
 		)
-		(property "Value" "0.1uF"
+		(property "Value" "100nF"
 			(at 0 1.43 0)
 			(layer "F.Fab")
@@
 			)
 		)
-		(property "Value" "0.1uF"
+		(property "Value" "100nF"
 			(at 0 1.43 0)
 			(layer "F.Fab")
@@
 			)
 		)
-		(property "Value" "0.1uF"
+		(property "Value" "100nF"
 			(at 0 1.43 0)
 			(layer "F.Fab")
@@
 			)
 		)
+		(attr exclude_from_bom)
 		(duplicate_pad_numbers_are_jumpers no)
 		(fp_circle
@@
 			)
 		)
-		(property "Value" "0.1uF"
+		(property "Value" "100nF"
 			(at 0 -1.43 90)
 			(layer "B.Fab")
@@
 			)
 		)
-		(property "Value" "0.1uF"
+		(property "Value" "100nF"
 			(at 0 -1.43 90)
 			(layer "B.Fab")
@@
 			)
 		)
-		(property "Value" "0.1uF"
+		(property "Value" "100nF"
 			(at 0 -1.43 0)
 			(layer "B.Fab")
@@
 			)
 		)
-		(property "LCSC" ""
+		(property "LCSC" "C22548"
 			(at 0 0 180)
 			(unlocked yes)
@@
 			)
 		)
+		(attr exclude_from_bom)
 		(duplicate_pad_numbers_are_jumpers no)
 		(fp_circle
@@
 			)
 		)
-		(property "LCSC" ""
+		(property "LCSC" "C22548"
 			(at 0 0 270)
 			(unlocked yes)
@@
 			)
 		)
-		(property "Value" "0.1uF"
+		(property "Value" "100nF"
 			(at 0 -1.43 0)
 			(layer "B.Fab")
@@
 			)
 		)
-		(property "LCSC" ""
+		(property "LCSC" "C22548"
 			(at 0 0 180)
 			(unlocked yes)
@@
 			)
 		)
+		(attr exclude_from_bom)
 		(duplicate_pad_numbers_are_jumpers no)
 		(fp_circle
@@
 			)
 		)
-		(property "Value" "0.1uF"
+		(property "Value" "100nF"
 			(at 0 -1.43 0)
 			(layer "B.Fab")
@@
 			)
 		)
+		(attr exclude_from_bom)
 		(duplicate_pad_numbers_are_jumpers no)
 		(fp_circle
@@
 			)
 		)
-		(property "Value" "0.1uF"
+		(property "Value" "100nF"
 			(at 0 -1.43 0)
 			(layer "B.Fab")
@@
 			)
 		)
+		(attr exclude_from_bom)
 		(duplicate_pad_numbers_are_jumpers no)
 		(fp_circle
@@
 			)
 		)
+		(attr exclude_from_bom)
 		(duplicate_pad_numbers_are_jumpers no)
 		(fp_circle
@@
 			)
 		)
+		(attr exclude_from_bom)
 		(duplicate_pad_numbers_are_jumpers no)
 		(fp_circle
@@
 			)
 		)
-		(property "Value" "0.1uF"
+		(property "Value" "100nF"
 			(at 0 -1.43 90)
 			(layer "B.Fab")
@@
 			)
 		)
-		(property "LCSC" ""
+		(property "LCSC" "C22548"
 			(at 0 0 270)
 			(unlocked yes)
@@
 			)
 		)
-		(property "LCSC" ""
+		(property "LCSC" "C22548"
 			(at 0 0 180)
 			(unlocked yes)
@@
 			)
 		)
-		(property "LCSC" ""
+		(property "LCSC" "C22548"
 			(at 0 0 180)
 			(unlocked yes)
@@
 			)
 		)
-		(property "LCSC" ""
+		(property "LCSC" "C22548"
 			(at 0 0 270)
 			(unlocked yes)
@@
 			)
 		)
-		(property "Value" "0.1uF"
+		(property "Value" "100nF"
 			(at 0 -1.43 90)
 			(layer "B.Fab")
@@
 			)
 		)
-		(property "LCSC" ""
+		(property "LCSC" "C22548"
 			(at 0 0 270)
 			(unlocked yes)
@@
 			)
 		)
-		(property "Part Number" "MI0603K300R-10"
+		(property "Part Number" "FCM1608KF-601T05"
 			(at 0 0 270)
 			(unlocked yes)
@@
 			)
 		)
-		(property "LCSC" "C96708"
+		(property "LCSC" "C133937"
 			(at 0 0 90)
 			(unlocked yes)
@@
 			)
 		)
+		(attr exclude_from_bom)
 		(duplicate_pad_numbers_are_jumpers no)
 		(fp_circle
@@
 		(width 0.3)
 		(layer "B.Cu")
-		(net "+12V")
-	)
-	(segment
-		(start 134.899948 84.2)
-		(end 134.899948 84.75)
-		(width 0.3)
-		(layer "B.Cu")
