File: hardware/motherboard/motherboard.kicad_pcb (KiCad board)
At the start: 4 copper layers, 150 x 90 mm, 28 parts, among them J1 Custom_PCIe_x4, J10 Conn_01x50_MountingPin, J11 Conn_01x50_MountingPin, J12 Barrel_Jack_Switch_Pin3Ring, J2 Custom_PCIe_x4, J3 Custom_PCIe_x4, J4 Custom_PCIe_x4, J5 Custom_PCIe_x4, J6 Custom_PCIe_x4, J7 Custom_PCIe_x4, J8 Custom_PCIe_x4, J9 Conn_01x50_MountingPin, U1 74HC138, U2 TMUX1208PW, U3 SN74LV595, U5 74HC138

Commit message: upldated
Parts:
- removed GND: TestPoint_Plated_Hole_D2.0mm, TestPoint:TestPoint_Plated_Hole_D2.0mm
- added C4: 0.1uF, Capacitor_SMD:C_0603_1608Metric, F.Cu at (158.8, 111.8)
- moved U2 77.1 mm to (163.0, 114.8), turned to 90 degrees
Connections:
- A1 pad 12: unconnected-(A1-GPIO9-Pad12) -> AT_EN
- A1 pad 17: unconnected-(A1-GPIO13-Pad17) -> TMUX
- J1 pad A3: +12V -> GND
- J1 pad A30: unconnected-(J1-RSVD-PadA30) -> +12V
- J1 pad A7: GND -> AT_1
- J2 pad A3: +12V -> GND
- J2 pad A30: unconnected-(J2-RSVD-PadA30) -> +12V
- J2 pad A7: GND -> AT_2
- J3 pad A3: +12V -> GND
- J3 pad A30: unconnected-(J3-RSVD-PadA30) -> +12V
- J3 pad A7: GND -> AT_3
- J4 pad A3: +12V -> GND
- J4 pad A30: unconnected-(J4-RSVD-PadA30) -> +12V
- J4 pad A7: GND -> AT_4
- J5 pad A3: +12V -> GND
- J5 pad A30: unconnected-(J5-RSVD-PadA30) -> +12V
- J5 pad A7: GND -> AT_5
- J6 pad A3: +12V -> GND
- J6 pad A30: unconnected-(J6-RSVD-PadA30) -> +12V
- J6 pad A7: GND -> AT_6
- J7 pad A3: +12V -> GND
- J7 pad A30: unconnected-(J7-RSVD-PadA30) -> +12V
- J7 pad A7: GND -> AT_7
- J8 pad A3: +12V -> GND
- J8 pad A30: unconnected-(J8-RSVD-PadA30) -> +12V
- J8 pad A7: GND -> AT_8
- U2 pad 1: unconnected-(U2-A0-Pad1) -> A1
- U2 pad 10: unconnected-(U2-S7-Pad10) -> AT_7
- U2 pad 11: unconnected-(U2-S6-Pad11) -> AT_6
- U2 pad 12: unconnected-(U2-S5-Pad12) -> AT_5
- U2 pad 13: unconnected-(U2-VDD-Pad13) -> +3.3V
- U2 pad 14: unconnected-(U2-GND-Pad14) -> GND
- U2 pad 15: unconnected-(U2-A2-Pad15) -> A3
- U2 pad 16: unconnected-(U2-A1-Pad16) -> A2
- U2 pad 2: unconnected-(U2-EN-Pad2) -> AT_EN
- U2 pad 3: unconnected-(U2-VSS-Pad3) -> GND
- U2 pad 4: unconnected-(U2-S1-Pad4) -> AT_1
- U2 pad 5: unconnected-(U2-S2-Pad5) -> AT_2
- U2 pad 6: unconnected-(U2-S3-Pad6) -> AT_3
- U2 pad 7: unconnected-(U2-S4-Pad7) -> AT_4
- U2 pad 8: unconnected-(U2-D-Pad8) -> TMUX
- U2 pad 9: unconnected-(U2-S8-Pad9) -> AT_8
Routing:
- net +3.3V: track 390.8 -> 200.9 mm, vias 14 -> 4
- net MOSI_1: track 209.0 -> 43.9 mm, vias 7 -> 3
- net CP: track 277.9 -> 125.7 mm, vias 14 -> 2
- net MISO_0: track 152.7 -> 5.88 mm, vias 15 -> 0
- net SCK_0: track 167.7 -> 22.8 mm, vias 4 -> 1
- net MOSI_0: track 173.6 -> 29.2 mm, vias 2 -> 1
- net SCK_1: track 157.4 -> 13.3 mm, vias 2 -> 1
- net PL: track 276.1 -> 137.4 mm, vias 14 -> 2
- net A2: track 88.0 -> 144.1 mm, vias 4 -> 8
- net +12V: track 214.3 -> 167.0 mm, vias 8 -> 7
- net A3: track 87.3 -> 123.3 mm, vias 5 -> 6
- net ADC_CS7: track 58.6 -> 31.5 mm
- net XTR_OD_7: track 49.1 -> 23.5 mm
- net XTR_OD_8: track 65.9 -> 41.6 mm
- net ADC_CS8: track 78.2 -> 56.3 mm
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