File: hardware/motherboard/motherboard.kicad_pcb (KiCad board)
At the start: 4 copper layers, 150 x 90 mm, 27 parts, among them J1 Custom_PCIe_x4, J10 Conn_01x50_MountingPin, J11 Conn_01x50_MountingPin, J12 Barrel_Jack_Switch_Pin3Ring, J2 Custom_PCIe_x4, J3 Custom_PCIe_x4, J4 Custom_PCIe_x4, J5 Custom_PCIe_x4, J6 Custom_PCIe_x4, J7 Custom_PCIe_x4, J8 Custom_PCIe_x4, J9 Conn_01x50_MountingPin, U1 74HC138, U3 SN74LV595, U5 74HC138

Commit message: updated daughterboard with eeprom and some layout improvements and padne simulations
Parts:
- added U2: TMUX1208PW, Package_SO:TSSOP-16_4.4x5mm_P0.65mm, F.Cu at (240.1, 113.1)
Connections:
- A1 pad 10: unconnected-(A1-GPIO7-Pad10) -> XTR_RCLK
- A1 pad 36: +3.3V -> unconnected-(A1-3V3-Pad36)
Routing:
- net XTR_RCLK: track 0.00 -> 74.1 mm, vias 0 -> 2
- net +3.3V: track 418.3 -> 390.8 mm, vias 15 -> 14
- net GND: vias 88 -> 86

Commit message: update pcb
Parts:
- removed GND: TestPoint_Plated_Hole_D2.0mm, TestPoint:TestPoint_Plated_Hole_D2.0mm
- added C4: 0.1uF, Capacitor_SMD:C_0603_1608Metric, F.Cu at (156.9, 112.0)
- added TP1: TestPoint, Connector_PinHeader_2.54mm:PinHeader_1x01_P2.54mm_Vertical, F.Cu at (240.6, 102.6)
- added TP2: TestPoint, Connector_PinHeader_2.54mm:PinHeader_1x01_P2.54mm_Vertical, F.Cu at (240.6, 107.2)
- added TP3: TestPoint, Connector_PinHeader_2.54mm:PinHeader_1x01_P2.54mm_Vertical, F.Cu at (240.6, 111.8)
- added TP4: TestPoint, Connector_PinHeader_2.54mm:PinHeader_1x01_P2.54mm_Vertical, F.Cu at (240.6, 116.4)
- moved U2 78.9 mm to (161.2, 115.0), turned to 90 degrees
- moved J6 3.57 mm to (130.5, 76.8)
- moved J5 3.54 mm to (148.5, 76.8)
- moved J1 3.33 mm to (220.8, 76.8)
- moved J4 3.30 mm to (166.6, 76.8)
- moved J8 3.29 mm to (94.3, 76.8)
- moved J7 3.28 mm to (112.4, 76.8)
- moved J3 3.24 mm to (184.7, 76.8)
- moved J2 3.23 mm to (202.8, 76.8)
Connections:
- A1 pad 12: unconnected-(A1-GPIO9-Pad12) -> AT_EN
- A1 pad 16: unconnected-(A1-GPIO12-Pad16) -> MISO_1
- A1 pad 17: unconnected-(A1-GPIO13-Pad17) -> AT_MUX
- J1 pad A3: +12V -> GND
- J1 pad A30: unconnected-(J1-RSVD-PadA30) -> +12V
- J1 pad A7: GND -> AT1
- J1 pad B9: +3.3V -> MISO_1
- J2 pad A3: +12V -> GND
- J2 pad A30: unconnected-(J2-RSVD-PadA30) -> +12V
- J2 pad A7: GND -> AT2
- J2 pad B9: +3.3V -> MISO_1
- J3 pad A3: +12V -> GND
- J3 pad A30: unconnected-(J3-RSVD-PadA30) -> +12V
- J3 pad A7: GND -> AT3
- J3 pad B9: +3.3V -> MISO_1
- J4 pad A3: +12V -> GND
- J4 pad A30: unconnected-(J4-RSVD-PadA30) -> +12V
- J4 pad A7: GND -> AT4
- J4 pad B9: +3.3V -> MISO_1
- J5 pad A3: +12V -> GND
- J5 pad A30: unconnected-(J5-RSVD-PadA30) -> +12V
- J5 pad A7: GND -> AT5
- J5 pad B9: +3.3V -> MISO_1
- J6 pad A3: +12V -> GND
- J6 pad A30: unconnected-(J6-RSVD-PadA30) -> +12V
- J6 pad A7: GND -> AT6
- J6 pad B9: +3.3V -> MISO_1
- J7 pad A3: +12V -> GND
- J7 pad A30: unconnected-(J7-RSVD-PadA30) -> +12V
- J7 pad A7: GND -> AT7
- J7 pad B9: +3.3V -> MISO_1
- J8 pad A3: +12V -> GND
- J8 pad A30: unconnected-(J8-RSVD-PadA30) -> +12V
- J8 pad A7: GND -> AT8
- J8 pad B9: +3.3V -> MISO_1
- U2 pad 1: unconnected-(U2-A0-Pad1) -> A1
- U2 pad 10: unconnected-(U2-S7-Pad10) -> AT7
- U2 pad 11: unconnected-(U2-S6-Pad11) -> AT6
- U2 pad 12: unconnected-(U2-S5-Pad12) -> AT5
- U2 pad 13: unconnected-(U2-VDD-Pad13) -> +3.3V
- U2 pad 14: unconnected-(U2-GND-Pad14) -> GND
- U2 pad 15: unconnected-(U2-A2-Pad15) -> A3
- U2 pad 16: unconnected-(U2-A1-Pad16) -> A2
- U2 pad 2: unconnected-(U2-EN-Pad2) -> AT_EN
- U2 pad 3: unconnected-(U2-VSS-Pad3) -> GND
- U2 pad 4: unconnected-(U2-S1-Pad4) -> AT1
- U2 pad 5: unconnected-(U2-S2-Pad5) -> AT2
- U2 pad 6: unconnected-(U2-S3-Pad6) -> AT3
- U2 pad 7: unconnected-(U2-S4-Pad7) -> AT4
- U2 pad 8: unconnected-(U2-D-Pad8) -> AT_MUX
- U2 pad 9: unconnected-(U2-S8-Pad9) -> AT8
Routing:
- net +3.3V: track 390.8 -> 184.9 mm, vias 14 -> 0
- net MISO_1: track 0.00 -> 177.8 mm, vias 0 -> 8
- net CP: track 277.9 -> 133.0 mm, vias 14 -> 0
- net PL: track 276.1 -> 133.7 mm, vias 14 -> 0
- net Q7_8: track 139.6 -> 0.00 mm, vias 3 -> 0
- net DAC_CS1: track 108.6 -> 3.11 mm, vias 4 -> 0
- net XTR_OD_1: track 114.2 -> 9.73 mm, vias 3 -> 0
- net ADC_CS1: track 108.7 -> 6.80 mm, vias 3 -> 0
- net XTR_OD_2: track 99.1 -> 0.00 mm, vias 1 -> 0
- net DAC_EN: track 98.0 -> 0.00 mm, vias 4 -> 0
- net XTR_OD_3: track 84.8 -> 0.00 mm, vias 1 -> 0
- net +12V: track 214.3 -> 132.0 mm, vias 8 -> 0
- net ADC_CS2: track 80.4 -> 0.00 mm, vias 3 -> 0
- net DAC_CS2: track 80.2 -> 0.00 mm, vias 4 -> 0
- net ADC_CS8: track 78.2 -> 0.00 mm, vias 3 -> 0
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Other:
- board text removed: "1"
- board text removed: "2"
- board text removed: "3"
- board text removed: "4"
- board text removed: "5"
- board text removed: "6"
- board text removed: "7"
- board text removed: "8"
