File: hardware/motherboard/motherboard.kicad_pcb (KiCad board)
At the start: 4 copper layers, 150 x 90 mm, 40 parts, among them J1 PCIE-064-02-F-D-TH, J10 Conn_01x50_MountingPin, J11 Conn_01x50_MountingPin, J12 Barrel_Jack_Switch_Pin3Ring, J2 PCIE-064-02-F-D-TH, J3 PCIE-064-02-F-D-TH, J4 PCIE-064-02-F-D-TH, J5 PCIE-064-02-F-D-TH, J6 PCIE-064-02-F-D-TH, J7 PCIE-064-02-F-D-TH, J8 PCIE-064-02-F-D-TH, J9 Conn_01x50_MountingPin, Q1 AO3407A, U1 SN74HC138PWR, U2 TMUX1208PW, U3 SN74LV595, U4 LP5912-3.3DRV, U5 SN74HC138PWR, U6 K7805-500R3

Commit message: routed
Routing:
- net CH40: track 2.50 -> 50.4 mm
- net CH41: track 2.50 -> 46.6 mm
- net CH16: track 2.50 -> 45.1 mm
- net CH0: track 2.50 -> 43.3 mm
- net CH17: track 2.50 -> 43.3 mm
- net CH32: track 2.50 -> 41.8 mm
- net CH56: track 2.50 -> 41.7 mm
- net CH24: track 2.50 -> 41.0 mm
- net CH42: track 6.50 -> 44.4 mm
- net CH1: track 2.50 -> 40.4 mm
- net CH48: track 2.50 -> 39.8 mm
- net CH57: track 2.50 -> 39.3 mm
- net CH33: track 2.50 -> 39.1 mm
- net CH25: track 2.50 -> 38.8 mm
- net CH18: track 6.50 -> 42.6 mm
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