File: hardware/motherboard/motherboard.kicad_sch (KiCad schematic)
At the start: 21 parts, among them J1 Custom_PCIe_x4, J10 Conn_01x50_MountingPin, J11 Conn_01x50_MountingPin, J12 Barrel_Jack_Switch_Pin3Ring, J2 Custom_PCIe_x4, J3 Custom_PCIe_x4, J4 Custom_PCIe_x4, J5 Custom_PCIe_x4, J6 Custom_PCIe_x4, J7 Custom_PCIe_x4, J8 Custom_PCIe_x4, J9 Conn_01x50_MountingPin, U1 74HC138, U2 TMUX1208PW, U3 SN74LV595, U5 74HC138

Commit message: upldated
Parts:
- added C4: 0.1uF, Capacitor_SMD:C_0603_1608Metric, symbol Device:C_Small
Connections:
- net +12V: now also J1.A30 (+12V), J2.A30 (+12V), J3.A30 (+12V), J4.A30 (+12V), J5.A30 (+12V), J6.A30 (+12V), J7.A30 (+12V), J8.A30 (+12V); no longer J1.A3 (+3.3V), J2.A3 (+3.3V), J3.A3 (+3.3V), J4.A3 (+3.3V), J5.A3 (+3.3V), J6.A3 (+3.3V), J7.A3 (+3.3V), J8.A3 (+3.3V)
- net +3.3V: now also U2.13 (VDD), C4.1
- net GND: now also J1.A3 (GND), J2.A3 (GND), J3.A3 (GND), J4.A3 (GND), J5.A3 (GND), J6.A3 (GND), J7.A3 (GND), J8.A3 (GND), U2.14 (GND), U2.3 (VSS), C4.2; no longer J1.A7 (GND), J2.A7 (GND), J3.A7 (GND), J4.A7 (GND), J5.A7 (GND), J6.A7 (GND), J7.A7 (GND), J8.A7 (GND)
- net TMUX: now reaches A1.17 (GPIO13)
- net TMUX: now also U2.8 (D)
- net AT_7: now reaches U2.10 (S7)
- net AT_7: now also J7.A7 (AT)
- net AT_6: now reaches U2.11 (S6)
- net AT_6: now also J6.A7 (AT)
- net AT_5: now reaches U2.12 (S5)
- net AT_5: now also J5.A7 (AT)
- net AT_1: now reaches U2.4 (S1)
- net AT_1: now also J1.A7 (AT)
- net AT_2: now reaches U2.5 (S2)
- net AT_2: now also J2.A7 (AT)
- net AT_3: now reaches U2.6 (S3)
- net AT_3: now also J3.A7 (AT)
- net AT_4: now reaches U2.7 (S4)
- net AT_4: now also J4.A7 (AT)
- net AT_8: now reaches U2.9 (S8)
- net AT_8: now also J8.A7 (AT)
- no-connect marks 45 -> 37
