File: hardware/motherboard/motherboard.kicad_sch (KiCad schematic)
At the start: 26 parts, among them J1 Custom_PCIe_x4, J10 Conn_01x50_MountingPin, J11 Conn_01x50_MountingPin, J12 Barrel_Jack_Switch_Pin3Ring, J2 Custom_PCIe_x4, J3 Custom_PCIe_x4, J4 Custom_PCIe_x4, J5 Custom_PCIe_x4, J6 Custom_PCIe_x4, J7 Custom_PCIe_x4, J8 Custom_PCIe_x4, J9 Conn_01x50_MountingPin, U1 74HC138, U2 TMUX1208PW, U3 SN74LV595, U5 74HC138

Commit message: Motherboard: protected power input, K7805 switcher, working 3V3_EN interlock
Rework the motherboard power tree from the barrel jack to the 3.3 V rail.
Design rationale and verification are recorded in hardware/motherboard/POWER.md.

Input protection (new):
- F1 PPTC 1.5 A hold / 3 A trip (1812L150/24MR) -> D2 SMBJ13A TVS -> Q1 AO3407A
  P-FET reverse-polarity, in that order so a surge or reversed jack crowbars
  through the fuse.
- Q1 is drain-to-supply / source-to-load; source-to-supply passes reverse
  current through the body diode and fails silently.
- AO3407A (Vgs +/-20 V) replaces AO3401A (+/-12 V), which sat at its absolute
  maximum on a 12 V rail and needed a gate zener conducting continuously.
- +12 V now actually reaches J1-J8 pin A30; it was previously an orphan net
  with no source.

Regulation:
- U8 L7805 -> K7805-500R3 switching module, pin-compatible with LM78xx.
  Cuts 12->5 V loss from ~1.5 W to ~0.15 W. TRACO TSR-1 symbol/footprint match
  the datasheet layout (3 x 1.00 mm holes, 2.54 mm pitch).
- Datasheet-required caps added: C5 10 uF/50 V at the input, C6 22 uF at the
  output, C7 220 uF electrolytic bulk for load steps and hot-plug damping.

3V3_EN interlock (was inert):
- R7 100k -> 10k, R8 100k -> 4.7k with its far end moved from the Pico's own
  3V3 output (pin 36) to the board +3.3 V rail. As wired it was a bootstrap
  divider off the regulator's own output that enabled in every case.
- Verified against RT6150A/B DS6150A/B-06: EN logic-low max 0.4 V, logic-high
  min 1.2 V. Board rail dead -> 0.146 V (off); rail up -> 2.32 V (on).

Also:
- U1/U5 SN74LVC138APWR -> SN74HC138PWR: 8x cheaper, ~50k stock vs 669, and
  the decoders are static during a transfer (address then enable, then SPI).
  Footprint corrected SSOP-16 -> TSSOP-16, matching the PW part and U2/U3.
- Capacitors standardised on 0805 (C8 stays 1210 for DC-bias reasons).
- Footprints assigned to F1/R1/R6/R7/R8; LCSC part numbers recorded in POWER.md.
- .gitignore: padne output, Ki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
Parts:
- removed PS1: DSM2-12-S3-S, Converter_DCDC:Converter_DCDC_XP_POWER-IAxxxxS_THT, symbol Converter_DCDC:IA0305S
- removed TP1, TP2, TP3, TP4: TestPoint, Connector_PinHeader_2.54mm:PinHeader_1x01_P2.54mm_Vertical, symbol Connector:TestPoint
- added C5: 10uF, Capacitor_SMD:C_1210_3225Metric, symbol Device:C_Small
- added C6: 22uF, Capacitor_SMD:C_0805_2012Metric, symbol Device:C_Small
- added C7: 220uF, Capacitor_SMD:CP_Elec_8x10, symbol Device:C_Polarized_Small
- added C8, C9: 10uF, Capacitor_SMD:C_0805_2012Metric, symbol Device:C_Small
- added D1: SS34, Diode_SMD:D_SMA, symbol Diode:SS34
- added D2: SMBJ13A, Diode_SMD:D_SMB, symbol Diode:SM6T68A
- added F1: 1812L150/24MR, Fuse:Fuse_1812_4532Metric, symbol Device:Polyfuse
- added Q1: AO3407A, Package_TO_SOT_SMD:SOT-23, symbol Transistor_FET:AO3401A
- added R1, R6: 100k, Resistor_SMD:R_0805_2012Metric, symbol Device:R_Small_US
- added R7: 10k, Resistor_SMD:R_0805_2012Metric, symbol Device:R_Small_US
- added R8: 4.7k, Resistor_SMD:R_0805_2012Metric, symbol Device:R_Small_US
- added U4: LP5912-3.3DRV, Package_SON:WSON-6-1EP_2x2mm_P0.65mm_EP1x1.6mm_ThermalVias, symbol Regulator_Linear:LP5912-3.3DRV
- added U6: K7805-500R3, Converter_DCDC:Converter_DCDC_TRACO_TSR-1_THT, symbol Converter_DCDC:TSR_1-2450
- C1, C2, C3, C4: LCSC (none) -> C14663
- J1, J2, J3, J4, J5, J6, J7, J8: value Custom_PCIe_x4 -> PCIE-064-02-F-D-TH; LCSC (none) -> C4597619
- J12: LCSC (none) -> C84007
- U1, U5: value 74HC138 -> SN74HC138PWR; footprint Package_SO:SSOP-16_5.3x6.2mm_P0.65mm -> Package_SO:TSSOP-16_4.4x5mm_P0.65mm; LCSC (none) -> C157527
- U2: LCSC (none) -> C494728
- U3: LCSC (none) -> C116847
Connections:
- net +12V: now also C5.1, C7.1, Q1.2 (S), U6.1 (Vin); no longer J12.1
- net +3.3V: now also U1.6 (E2), U5.6 (E2), C9.1, R6.1, R8.2, U4.1 (OUT)
- net GND: now also C5.2, C6.2, C7.2, C8.2, C9.2, D2.2 (A2), R1.2, R7.1, U4.5 (GND), U4.7 (EP), U6.2 (GND); no longer J1.B31 (~{PRSNT2}), J2.B31 (~{PRSNT2}), J3.B31 (~{PRSNT2}), J4.B31 (~{PRSNT2}), J5.B31 (~{PRSNT2}), J6.B31 (~{PRSNT2}), J7.B31 (~{PRSNT2}), J8.B31 (~{PRSNT2}), U1.6 (E2), U5.6 (E2)
- net PG: now reaches A1.11 (GPIO8)
- net PG: now also R6.2, U4.3 (PG)
- net 3V3_EN: now reaches A1.37 (3V3_EN)
- net 3V3_EN: now also R7.2, R8.1
- net VSYS: now reaches A1.39 (VSYS)
- net VSYS: now also D1.1 (K)
- new net: Q1.1 (G), R1.1
- new net: D2.1 (A1), F1.1, Q1.3 (D)
- new net +5V: C6.1, C8.1, D1.2 (A), U4.4 (EN), U4.6 (IN), U6.3 (Vout)
- new net PRSNT: J1.B31 (~{PRSNT2})
- new net VIN_JACK: F1.2, J12.1
- no-connect marks 36 -> 37
Other:
- note removed: "The Golden Rule for your Firmware Because of the AD7193's /WEN bit, you must clear the bus before selecting a new chip. Your C/C++ function for reading these ADCs must follow this exact rigid sequence: Assert: Pull 595 Latch LOW. Select: Send 11111110 (or whichever ADC you want). Lock: Pull 595 Latch HIGH. (Target ADC is now active). Communicate: Send your AD7193 command (starting with 0) and rea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"
- moved on the sheet: A1

Commit message: motherboard: protected input stage, 12->5->3.3 V tree, 3V3_EN interlock
Replaces PS1 with a staged supply and puts the Pico behind a hardware
interlock, per hardware/motherboard/POWER.md.

Input protection: F1 1812L150/24MR PPTC, D2 SMBJ13A TVS, Q1 AO3407A
reverse-polarity P-FET (R1 100k gate). Q1 source now sources +12V, which
previously reached J1-J8.A30 with no source at all.

Rails: U6 K7805-500R3 (12->5 V) replaces the L7805, feeding D1 SS34 to
the Pico VSYS and U4 LP5912-3.3 to the logic rail. Bulk and decoupling
sized to datasheet minimums (C5/C7 on +12V, C6/C8 on +5V, C1-C4/C9 on
+3.3V). D3/D4/D5 rail LEDs, J13 +12 V header.

3V3_EN interlock: R8 4.7k from the board +3.3V rail to A1 pin 37, R7 10k
to GND. Against the module's internal 100k pull-up to VSYS this holds
3V3_EN at ~0.15 V when the jack is absent, so the RP2040 cannot run on
USB power alone. A1 pins 36/40 stay unconnected.

Note this means the Pico cannot be flashed over USB without jack power.

BOM now carries LCSC numbers throughout; J9-J11 move to Hirose
FH12-50S-0.5SH (the Molex 54132-5033 was not stocked) and U2 TMUX1208PW
resolves to C494728, closing both open sourcing questions in POWER.md.

Co-Authored-By: Claude Opus 5 <noreply@anthropic.com>
Parts:
- added D3, D4, D5: LED, LED_SMD:LED_0603_1608Metric, symbol Device:LED
- added D6: BZT52Bxx, Diode_SMD:D_SOD-123F, symbol Diode:BZT52Bxx
- added FID1, FID2: Fiducial, Fiducial:Fiducial_0.75mm_Mask1.5mm, symbol Mechanical:Fiducial
- added J13: Conn_01x02_Pin, Connector_PinHeader_2.54mm:PinHeader_1x02_P2.54mm_Vertical, symbol Connector:Conn_01x02_Pin
- added R2: 4.7k, Resistor_SMD:R_0805_2012Metric, symbol Device:R_Small_US
- added R3: 1.5k, Resistor_SMD:R_0805_2012Metric, symbol Device:R_Small_US
- added R4: 680, Resistor_SMD:R_0805_2012Metric, symbol Device:R_Small_US
- added R9: 10k, Resistor_SMD:R_0805_2012Metric, symbol Device:R_Small_US
- A1: LCSC (none) -> C7203003
- J10, J11, J9: footprint Connector_FFC-FPC:Molex_54132-5033_1x50-1MP_P0.5mm_Horizontal -> Connector_FFC-FPC:Hirose_FH12-50S-0.5SH_1x50-1MP_P0.50mm_Horizontal; LCSC (none) -> C202116
- R8: LCSC C60816 -> C431850
Connections:
- net PRSNT is gone; now on net GND: J1.B31 (~{PRSNT2})
- net +12V: now also D3.2 (A), D6.1 (K), J13.1 (Pin_1)
- net +3.3V: now also D5.2 (A), R9.2
- net +5V: now also D4.2 (A)
- net GND: now also J2.B31 (~{PRSNT2}), J3.B31 (~{PRSNT2}), J4.B31 (~{PRSNT2}), J5.B31 (~{PRSNT2}), J6.B31 (~{PRSNT2}), J7.B31 (~{PRSNT2}), J13.2 (Pin_2), R2.1, R3.1, R4.1; no longer U3.13 (~{OE})
- net ~{OE}: now reaches A1.25 (GPIO19)
- net ~{OE}: now also U3.13 (~{OE}), R9.1
- net at Q1.1 (G), R1.1: now also D6.2 (A)
- new net: D4.1 (K), R3.2
- new net: D5.1 (K), R4.2
- new net: D3.1 (K), R2.2
- no-connect marks 37 -> 36
Other:
- moved on the sheet: C5, C6, C7, C8, C9, D1, D2, F1, J12, Q1, R1, R6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

Commit message: hardware: release both boards to fabrication
Fab outputs regenerated from the current designs and sent out 2026-08-12.

Motherboard:
- +12V sense divider R5/R10 (100k/22k) + C10 filter at the Pico ADC pin
  -> GPIO26/ADC0, ratio 0.1803
- U3.~OE cut over from hardwired GND to GPIO19 (R9 10k pull-up)
- D2 SMBJ13A -> SMBJ16A (13 V standoff conducts on a 15 V rail)
- D6 gate-source clamp fixed at BZT52C18 (C192739)
- J1..J8.B31 tied to GND on all eight; dangling one-node PRSNT net deleted

Daughterboard:
- 1k series resistors R28-R35 into the OPA2333 followers
- L1 ferrite requoted C96708 (delisted) -> C133937, same 600R@100MHz
- U10 REF5030IDGKR -> REF5030EIDR; test points and the card edge J1 taken
  out of the BOM (bare pads / edge fingers, not parts)

master_bom.csv: D2 requote, D6/C10/R5/R10 added, L1 priced; $709.08 -> $709.29.
POWER.md: production/ is no longer stale (it is the released set); the two
remaining open items are schematic-drawing hygiene, not connectivity.
README: status section reflects the boards being in fab.

Co-Authored-By: Claude Opus 5 <noreply@anthropic.com>
Parts:
- added C10: 0.1uF, Capacitor_SMD:C_0603_1608Metric, symbol Device:C_Small
- added R10: 22k, Resistor_SMD:R_0805_2012Metric, symbol Device:R_Small_US
- added R5: 100k, Resistor_SMD:R_0805_2012Metric, symbol Device:R_Small_US
- D2: value SMBJ13A -> SMBJ16A; LCSC C133675 -> C151254
- D6: value BZT52Bxx -> BZT52C18; footprint Diode_SMD:D_SOD-123F -> Diode_SMD:D_SOD-123; LCSC (none) -> C192739
- J13: LCSC (none) -> C32713268
Connections:
- net +12V: now also R5.1
- net GND: now also J8.B31 (~{PRSNT2}), C10.2, R10.2
- net 12V_SENSE: now reaches A1.31 (GPIO26_ADC0)
- net 12V_SENSE: now also C10.1, R10.1, R5.2
- no-connect marks 36 -> 35
Other:
- note removed: "maybe move the power pins"
- moved on the sheet: D1
